File: hw/micromod_adapter/MicroMod_ATP_CarrierBoard.kicad_sch (KiCad schematic)
At the start: 70 parts, among them J1 USB_C_2-LAYER_PADS, J10 CONN_05VERT_FEMALE_HEADER, J11 CONN_041X04_NO_SILK_NO_POP, J12 CONN_12SMD_COMBINED, J13 CONN_08NO_SILK_DNP, J14 CONN_08SMD-COMBO-FEMALE, J15 CONN_08NO_SILK_FEMALE_PTH, J16 CONN_041X04_NO_SILK_NO_POP, J17 CONN_08SMD-COMBO-FEMALE, J18 CONN_08NO_SILK_FEMALE_PTH, J19 QWIIC_RIGHT_ANGLE, J2 JTAG, J20 QWIIC_RIGHT_ANGLE, J21 1X04_SMD_STRAIGHT_COMBO, J22 CONN_041X04_NO_SILK_NO_POP, J23 CONN_08NO_SILK_FEMALE_PTH, J24 CONN_08SMD-COMBO-FEMALE, J25 CONN_08SMD-COMBO-FEMALE, J26 CONN_08NO_SILK_FEMALE_PTH, J3 CONN_05NO_SILK, J4 USB_A_SMT_FEMALE, J6 MICROMOD-2222-C, J8 1X04_SMD_STRAIGHT_COMBO, J9 CONN_041X04_NO_SILK, U5 AP7361C-33

Commit message: updates
Parts:
- removed J10: CONN_05VERT_FEMALE_HEADER, 1X05_SMD_VERTICAL_COMBO, symbol MicroMod_ATP_CarrierBoard-eagle-import:CONN_05VERT_FEMALE_HEADER
- removed J12: CONN_12SMD_COMBINED, 1X12_SMD_COMBINED, symbol MicroMod_ATP_CarrierBoard-eagle-import:CONN_12SMD_COMBINED
- removed J13: CONN_08NO_SILK_DNP, 1X08_NO_SILK, symbol MicroMod_ATP_CarrierBoard-eagle-import:CONN_08NO_SILK_DNP
- removed J14, J17, J24, J25: CONN_08SMD-COMBO-FEMALE, 1X08_SMD_COMBINED, symbol MicroMod_ATP_CarrierBoard-eagle-import:CONN_08SMD-COMBO-FEMALE
- removed J15, J18, J23, J26: CONN_08NO_SILK_FEMALE_PTH, 1X08_NO_SILK, symbol MicroMod_ATP_CarrierBoard-eagle-import:CONN_08NO_SILK_FEMALE_PTH
- removed J16, J22: CONN_041X04_NO_SILK_NO_POP, 1X04_NO_SILK, symbol MicroMod_ATP_CarrierBoard-eagle-import:CONN_041X04_NO_SILK_NO_POP
- removed J19, J20: QWIIC_RIGHT_ANGLE, JST04_1MM_RA, symbol MicroMod_ATP_CarrierBoard-eagle-import:QWIIC_CONNECTORJS-1MM
- removed J21, J8: 1X04_SMD_STRAIGHT_COMBO, 1X04_SMD_VERTICAL_COMBO, symbol MicroMod_ATP_CarrierBoard-eagle-import:CONN_04SMD_STRAIGHT_COMBO
- removed J3: CONN_05NO_SILK, 1X05_NO_SILK, symbol MicroMod_ATP_CarrierBoard-eagle-import:CONN_05NO_SILK
- removed J9: CONN_041X04_NO_SILK, 1X04_NO_SILK, symbol MicroMod_ATP_CarrierBoard-eagle-import:CONN_041X04_NO_SILK
- added J?: Raspberry_Pi_2_3, Connector_PinSocket_2.54mm:PinSocket_2x20_P2.54mm_Vertical, symbol Connector:Raspberry_Pi_2_3
Connections:
- net GND: now also J?.14 (GND), J?.20 (GND), J?.25 (GND), J?.30 (GND), J?.34 (GND), J?.39 (GND), J?.6 (GND), J?.9 (GND)
- net A0 renamed PI-ACT
- net PI-ACT: now also J?.7 (GCLK0/GPIO4)
- net A1 renamed DBG_LED
- net DBG_LED: now also J?.29 (GCLK1/GPIO5)
- net CAN_RXI renamed PI-IND
- net PI-IND: now also J?.31 (GCLK2/GPIO6)
- net CAN_TXO renamed PI-DTD
- net PI-DTD: now also J?.24 (~{CE0}/GPIO8)
- net G0 renamed PI-D0
- net PI-D0: now also J?.19 (MOSI0/GPIO10)
- net G1 renamed PI-D1
- net PI-D1: now also J?.23 (SCLK0/GPIO11)
- net G10/ADC_P renamed PI-RST
- net PI-RST: now also J?.38 (GPIO20/MOSI1)
- net G11 renamed PI-ACK
- net PI-ACK: now also J?.40 (GPIO21/SCLK1)
- net G2 renamed PI-D2
- net PI-D2: now also J?.32 (PWM0/GPIO12)
- net G3 renamed PI-D3
- net PI-D3: now also J?.33 (PWM1/GPIO13)
- net G4 renamed PI-D4
- net PI-D4: now also J?.8 (GPIO14/TXD)
- net G5 renamed PI-D5
- net PI-D5: now also J?.10 (GPIO15/RXD)
- net G6 renamed PI-D6
- net PI-D6: now also J?.36 (GPIO16)
- net G7 renamed PI-D7
- net PI-D7: now also J?.11 (GPIO17)
- net G8 renamed PI-DP
- net PI-DP: now also J?.12 (GPIO18/PWM0)
- net G9/ADC_N renamed PI-ATN
- net PI-ATN: now also J?.35 (GPIO19/MISO1)
- net I2C_~{INT} renamed PI_GPIO9
- net PI_GPIO9: now also J?.21 (MISO0/GPIO9)
- net I2S_CLK renamed PI-REQ
- net PI-REQ: now also J?.15 (GPIO22)
- net I2S_SDI renamed PI-C_D
- net PI-C_D: now also J?.18 (GPIO24)
- net I2S_SDO renamed PI-I_O
- net PI-I_O: now also J?.22 (GPIO25)
- net I2S_WS renamed PI-MSG
- net PI-MSG: now also J?.16 (GPIO23)
- net MCLK renamed PI-BSY
- net PI-BSY: now also J?.37 (GPIO26)
- net RX2 renamed PI-SEL
- net PI-SEL: now also J?.13 (GPIO27)
- net SCL renamed PI_SCL
- net PI_SCL: now also J?.5 (SCL/GPIO3)
- net SDA renamed PI_SDA
- net PI_SDA: now also J?.3 (SDA/GPIO2)
- net SWDCK renamed PI_GPIO1
- net PI_GPIO1: now also J?.28 (ID_SC/GPIO1)
- net SWDIO renamed PI_GPIO0
- net PI_GPIO0: now also J?.27 (ID_SD/GPIO0)
- net TX2 renamed PI-TAD
- net PI-TAD: now also J?.26 (~{CE1}/GPIO7)
- new net +3V3: J?.1 (3V3), J?.17 (3V3)
- new net +5V: J?.2 (5V), J?.4 (5V)
Other:
- note added: "Raspberry Pi Connector"

Commit message: did some stuff
Parts:
- removed C6: 0.1uF, 0603, symbol MicroMod_ATP_CarrierBoard-eagle-import:0.1UF-0603-25V-(+80/-20%)
- removed D1: 3.3V, SOD-323, symbol MicroMod_ATP_CarrierBoard-eagle-import:DIODE-ZENER-MM3Z3V3T1G
- removed FD1, FD2, FD3, FD4: FIDUCIALUFIDUCIAL, FIDUCIAL-MICRO, symbol MicroMod_ATP_CarrierBoard-eagle-import:FIDUCIALUFIDUCIAL
- removed H1, H2, H3, H4: STAND-OFF, STAND-OFF, symbol MicroMod_ATP_CarrierBoard-eagle-import:STAND-OFF
- removed J1: USB_C_2-LAYER_PADS, USB-C-16P-2LAYER-PADS, symbol MicroMod_ATP_CarrierBoard-eagle-import:USB_C_2-LAYER_PADS
- removed LOGO2: QWIIC_LOGO_5MM, QWIIC_5MM, symbol MicroMod_ATP_CarrierBoard-eagle-import:QWIIC_LOGO_5MM
- removed MEAS1: JUMPER-COMBO_2_NC_TRACE, COMBO-JUMPER_2_NC_TRACE, symbol MicroMod_ATP_CarrierBoard-eagle-import:JUMPER-COMBO_2_NC_TRACE
- removed R2, R3: 5.1k, 0603, symbol MicroMod_ATP_CarrierBoard-eagle-import:5.1KOHM5.1KOHM-0603-1/10W-1%
- removed R5: 100k, 0603, symbol MicroMod_ATP_CarrierBoard-eagle-import:100KOHM-0603-1/10W-1%
- removed TP1, TP2, TP3: TEST-POINT3X5, PAD.03X.05, symbol MicroMod_ATP_CarrierBoard-eagle-import:TEST-POINT3X5
- removed U5: AP7361C-33, UDFN-8, symbol MicroMod_ATP_CarrierBoard-eagle-import:AP7361C-33FGEUDFN-8
- added C6: 0.1uF, Capacitor_SMD:C_0805_2012Metric_Pad1.18x1.45mm_HandSolder, symbol Device:C_Small
- added H6, H7, H8, H9: MountingHole_Pad, MountingHole:MountingHole_2.7mm_M2.5_Pad_Via, symbol Mechanical:MountingHole_Pad
- added J1: U254-051N-4BH806, U254051N4BH806, symbol SamacSys_Parts:U254-051N-4BH806
- added J5: Conn_01x03_Male, Connector_PinHeader_2.54mm:PinHeader_1x03_P2.54mm_Vertical, symbol Connector:Conn_01x03_Male
- added J7: Conn_01x20_Male, Connector_PinHeader_1.00mm:PinHeader_1x24_P1.00mm_Vertical, symbol Connector:Conn_01x24_Male
- added R2: 0, Resistor_SMD:R_0805_2012Metric_Pad1.20x1.40mm_HandSolder, symbol Device:R_Small
- added U1: AMS1117-3.3, Package_TO_SOT_SMD:SOT-223-3_TabPin2, symbol Regulator_Linear:AMS1117-3.3
- 3V3_LED1, VIN_LED1: footprint SMT-JUMPER_2_NC_TRACE_SILK -> Jumper:SolderJumper-2_P1.3mm_Bridged_RoundedPad1.0x1.5mm; symbol MicroMod_ATP_CarrierBoard-eagle-import:JUMPER-SMT_2_NC_TRACE_SILK -> Jumper:SolderJumper_2_Bridged
- BYP1, EN1: footprint SMT-JUMPER_2_NO_SILK -> Jumper:SolderJumper-2_P1.3mm_Open_RoundedPad1.0x1.5mm; symbol MicroMod_ATP_CarrierBoard-eagle-import:JUMPER-SMT_2_NO_SILK -> Jumper:SolderJumper_2_Open
- C1: footprint 0603 -> Capacitor_SMD:C_0805_2012Metric_Pad1.18x1.45mm_HandSolder; symbol MicroMod_ATP_CarrierBoard-eagle-import:0.1UF-0603-25V-(+80/-20%) -> Device:C_Small; LCSC (none) -> C49678
- C13, C7: footprint 0603 -> Capacitor_SMD:C_0805_2012Metric_Pad1.18x1.45mm_HandSolder; symbol MicroMod_ATP_CarrierBoard-eagle-import:0.22UF-0603-25V-10% -> Device:C_Small; LCSC (none) -> C5378
- C2: footprint EIA3216 -> Capacitor_SMD:C_1206_3216Metric_Pad1.33x1.80mm_HandSolder; symbol MicroMod_ATP_CarrierBoard-eagle-import:10UF-POLAR-EIA3216-16V-10%(TANT) -> Device:C_Polarized_Small_US; LCSC (none) -> C7171
- C5: footprint 0603 -> Capacitor_SMD:C_0603_1608Metric_Pad1.08x0.95mm_HandSolder; symbol MicroMod_ATP_CarrierBoard-eagle-import:1.0UF-0603-16V-10% -> Device:C_Small; LCSC (none) -> C15849
- D2, D3: value RED -> Green; footprint LED-0603 -> LED_SMD:LED_0805_2012Metric_Pad1.15x1.40mm_HandSolder; symbol MicroMod_ATP_CarrierBoard-eagle-import:LED-RED0603 -> Device:LED_Small; LCSC (none) -> C2297
- R1, R4: footprint 0603 -> Capacitor_SMD:C_0805_2012Metric_Pad1.18x1.45mm_HandSolder; symbol MicroMod_ATP_CarrierBoard-eagle-import:1KOHM-0603-1/10W-1% -> Device:R_Small; LCSC (none) -> C17737
- R10: footprint 0603 -> Resistor_SMD:R_0805_2012Metric_Pad1.20x1.40mm_HandSolder; symbol MicroMod_ATP_CarrierBoard-eagle-import:20KOHM-0603-1/10W-1% -> Device:R_Small
- R9: footprint 0603 -> Resistor_SMD:R_0805_2012Metric_Pad1.20x1.40mm_HandSolder; symbol MicroMod_ATP_CarrierBoard-eagle-import:10KOHM-0603-1/10W-1% -> Device:R_Small; LCSC (none) -> C17414
- S1, S2: footprint TACTILE_SWITCH_SMD_5.2MM -> Button_Switch_THT:SW_PUSH_6mm
- gave numbers to parts that had none: 1
Connections:
- net 3.3V: now also C6.1, U1.2 (VO)
- net CIPO: now also J7.5 (Pin_5)
- net CIPO1/DAT0: now also J7.11 (Pin_11)
- net COPI: now also J7.6 (Pin_6)
- net COPI1: now also J7.10 (Pin_10)
- net CTS1: now also J7.15 (Pin_15)
- net D0: now also J7.20 (Pin_20)
- net D1: now also J7.19 (Pin_19)
- net DAT1: now also J7.12 (Pin_12)
- net DAT2: now also J7.13 (Pin_13)
- net GND: now also C2.2, C6.2, H6.1, H7.1, H8.1, H9.1, J1.5, J1.MH1, J1.MH2, J1.MH3, J1.MH4, J7.22 (Pin_22), J7.23 (Pin_23), J7.24 (Pin_24), R2.1, U1.1 (GND); no longer C2.-
- net PI_GPIO0: now also J5.2 (Pin_2)
- net PI_GPIO1: now also J5.3 (Pin_3)
- net PWM0: now also J7.2 (Pin_2)
- net PWM1: now also J7.3 (Pin_3)
- net RTC_3V: now also J5.1 (Pin_1)
- net RTS1: now also J7.16 (Pin_16)
- net RX1: now also J7.21 (Pin_21)
- net SCK: now also J7.7 (Pin_7)
- net SCK1: now also J7.9 (Pin_9)
- net SCL1: now also J7.18 (Pin_18)
- net SDA1: now also J7.17 (Pin_17)
- net TX1: now also J7.14 (Pin_14)
- net USB_N: now also J1.2
- net USB_P: now also J1.3
- net VIN: now also C2.1, U1.3 (VI); no longer C2.+
- net V_USB: now also J1.1
- net ~{CS1}/DAT3: now also J7.4 (Pin_4)
- net ~{CS}: now also J7.8 (Pin_8)
- net ~{RESET}: now also J7.1 (Pin_1)
- net at 3V3_LED1.1 (A): now also D2.1 (K); no longer D2.C
- net at R1.1: now also D2.2 (A); no longer D2.A
- net at VIN_LED1.1 (A): now also D3.1 (K); no longer D3.C
- net at R4.1: now also D3.2 (A); no longer D3.A
- new net: J1.4, R2.2
