File: hw/micromod_adapter/MicroMod_ATP_CarrierBoard.kicad_pcb (KiCad board)
At the start: 2 copper layers, 86.4 x 55.9 mm, 227 parts, among them J1 USB_C_2-LAYER_PADS, J10 CONN_05VERT_FEMALE_HEADER, J11 CONN_041X04_NO_SILK_NO_POP, J12 CONN_12SMD_COMBINED, J13 CONN_08NO_SILK_DNP, J14 CONN_08SMD-COMBO-FEMALE, J15 CONN_08NO_SILK_FEMALE_PTH, J16 CONN_041X04_NO_SILK_NO_POP, J17 CONN_08SMD-COMBO-FEMALE, J18 CONN_08NO_SILK_FEMALE_PTH, J19 QWIIC_RIGHT_ANGLE, J2 JTAG, J20 QWIIC_RIGHT_ANGLE, J21 1X04_SMD_STRAIGHT_COMBO, J22 CONN_041X04_NO_SILK_NO_POP, J23 CONN_08NO_SILK_FEMALE_PTH, J24 CONN_08SMD-COMBO-FEMALE, J25 CONN_08SMD-COMBO-FEMALE, J26 CONN_08NO_SILK_FEMALE_PTH, J3 CONN_05NO_SILK, J4 USB_A_SMT_FEMALE, J6 MICROMOD-2222-C, J8 1X04_SMD_STRAIGHT_COMBO, J9 CONN_041X04_NO_SILK, U5 AP7361C-33

Commit message: updates
Parts:
- removed 3V3_LED, VIN_LED: JUMPER-SMT_2_NC_TRACE_SILK, MicroMod_ATP_CarrierBoard:SMT-JUMPER_2_NC_TRACE_SILK
- removed BYP, EN: JUMPER-SMT_2_NO_SILK, MicroMod_ATP_CarrierBoard:SMT-JUMPER_2_NO_SILK
- removed H6, H7: STAND-OFF, MicroMod_ATP_CarrierBoard:STAND-OFF
- removed J10: CONN_05VERT_FEMALE_HEADER, MicroMod_ATP_CarrierBoard:1X05_SMD_VERTICAL_COMBO
- removed J12: CONN_12SMD_COMBINED, MicroMod_ATP_CarrierBoard:1X12_SMD_COMBINED
- removed J13: CONN_08NO_SILK_DNP, MicroMod_ATP_CarrierBoard:1X08_NO_SILK
- removed J14, J17, J24, J25: CONN_08SMD-COMBO-FEMALE, MicroMod_ATP_CarrierBoard:1X08_SMD_COMBINED
- removed J15, J18, J23, J26: CONN_08NO_SILK_FEMALE_PTH, MicroMod_ATP_CarrierBoard:1X08_NO_SILK
- removed J16, J22: CONN_041X04_NO_SILK_NO_POP, MicroMod_ATP_CarrierBoard:1X04_NO_SILK
- removed J19, J20: QWIIC_RIGHT_ANGLE, MicroMod_ATP_CarrierBoard:JST04_1MM_RA
- removed J21, J8: 1X04_SMD_STRAIGHT_COMBO, MicroMod_ATP_CarrierBoard:1X04_SMD_VERTICAL_COMBO
- removed J9: CONN_041X04_NO_SILK, MicroMod_ATP_CarrierBoard:1X04_NO_SILK
- removed LOGO4: SFE_LOGO_NAME_FLAME.2_INCH, MicroMod_ATP_CarrierBoard:SFE_LOGO_NAME_FLAME_.2
- removed LOGO5, LOGO6, LOGO7, LOGO8: QWIIC_LOGO_3MM, MicroMod_ATP_CarrierBoard:QWIIC_5MM
- removed MEAS: , MicroMod_ATP_CarrierBoard:COMBO-JUMPER_2_NC_TRACE
- removed U$1, U$123: , MicroMod_ATP_CarrierBoard:#A0#10
- removed U$10, U$116: , MicroMod_ATP_CarrierBoard:#G4#4
- removed U$100, U$101, U$102, U$103, U$104, U$105, U$27, U$3, U$46, U$47, U$58, U$89: , MicroMod_ATP_CarrierBoard:#GND#0
- removed U$106, U$107, U$126, U$38, U$60, U$61, U$70, U$88: , MicroMod_ATP_CarrierBoard:#3V3#1
- removed U$108, U$44: , MicroMod_ATP_CarrierBoard:#SDA#4
- removed U$109, U$49: , MicroMod_ATP_CarrierBoard:#SCL#5
- removed U$11, U$115: , MicroMod_ATP_CarrierBoard:#G5#5
- removed U$110, U$21: , MicroMod_ATP_CarrierBoard:##I2C_INT##10
- removed U$111, U$17: , MicroMod_ATP_CarrierBoard:#G11#10
- removed U$112, U$14: , MicroMod_ATP_CarrierBoard:#G8#8
- removed U$113, U$13: , MicroMod_ATP_CarrierBoard:#G7#7
- removed U$114, U$12: , MicroMod_ATP_CarrierBoard:#G6#6
- removed U$117, U$9: , MicroMod_ATP_CarrierBoard:#G3#3
- removed U$118, U$8: , MicroMod_ATP_CarrierBoard:#G2#2
- removed U$119, U$7: , MicroMod_ATP_CarrierBoard:#G1#2
- removed U$120, U$4: , MicroMod_ATP_CarrierBoard:#G0#2
- removed U$121, U$18: , MicroMod_ATP_CarrierBoard:#PWM0#10
- removed U$122, U$19: , MicroMod_ATP_CarrierBoard:#PWM1#10
- removed U$124, U$2: , MicroMod_ATP_CarrierBoard:#A1#10
- removed U$125, U$37: , MicroMod_ATP_CarrierBoard:##RESET##7
- removed U$127, U$45: , MicroMod_ATP_CarrierBoard:#VIN#6
- removed U$128, U$40: , MicroMod_ATP_CarrierBoard:#HOST_D##9
- removed U$129, U$41: , MicroMod_ATP_CarrierBoard:#HOST_D##10
- removed U$131, U$51: , MicroMod_ATP_CarrierBoard:#SWD#10
- removed U$132, U$42: , MicroMod_ATP_CarrierBoard:#MEAS#10
- removed U$133: , MicroMod_ATP_CarrierBoard:#VIN_LED#10
- removed U$134: , MicroMod_ATP_CarrierBoard:#3V3_LED#10
- removed U$135: , MicroMod_ATP_CarrierBoard:#G9#ADC##CAM_HSYNC#9
- removed U$136: , MicroMod_ATP_CarrierBoard:#G10#ADC##CAM_VSYNC#10
- removed U$137: , MicroMod_ATP_CarrierBoard:#I2S_SDI#CAM_PCLK#7
- removed U$138: , MicroMod_ATP_CarrierBoard:#I2S_SDO#CAM_MCLK#7
- removed U$139, U$141, U$142, U$143: , MicroMod_ATP_CarrierBoard:MOUNT10
- removed U$140: , MicroMod_ATP_CarrierBoard:MICROMOD_MI_LOGO_1
- removed U$144: , MicroMod_ATP_CarrierBoard:MICROMOD_LOGO_1
- removed U$145, U$99: , MicroMod_ATP_CarrierBoard:D10
- removed U$146, U$50: , MicroMod_ATP_CarrierBoard:#VHOST#0
- removed U$147: , MicroMod_ATP_CarrierBoard:#CIPO#5178038
- removed U$15: , MicroMod_ATP_CarrierBoard:#G9#9
- removed U$16: , MicroMod_ATP_CarrierBoard:#G10#10
- removed U$20: , MicroMod_ATP_CarrierBoard:##CS1##5178039
- removed U$22: , MicroMod_ATP_CarrierBoard:#CAN_RX#9
- removed U$23, U$97: , MicroMod_ATP_CarrierBoard:#CAN_TX#10
- removed U$24: , MicroMod_ATP_CarrierBoard:#CIPO#3
- removed U$25: , MicroMod_ATP_CarrierBoard:#COPI#2
- removed U$26: , MicroMod_ATP_CarrierBoard:#CTS#6
- removed U$28: , MicroMod_ATP_CarrierBoard:#SCK#2
- removed U$29: , MicroMod_ATP_CarrierBoard:#I2S_FS#5
- removed U$30: , MicroMod_ATP_CarrierBoard:#I2S_SDI#5
- removed U$31: , MicroMod_ATP_CarrierBoard:#I2S_SDO#5
- removed U$32: , MicroMod_ATP_CarrierBoard:#MCLK#4
- removed U$33: , MicroMod_ATP_CarrierBoard:#RTS#5
- removed U$34: , MicroMod_ATP_CarrierBoard:#RX#8
- removed U$35: , MicroMod_ATP_CarrierBoard:#TX#7
- removed U$36: , MicroMod_ATP_CarrierBoard:#DAT1#5178039
- removed U$39: , MicroMod_ATP_CarrierBoard:#BYP#8
- removed U$43: , MicroMod_ATP_CarrierBoard:BOOT10
- removed U$48: , MicroMod_ATP_CarrierBoard:#EN#0
- removed U$5: , MicroMod_ATP_CarrierBoard:#RESET10
- removed U$52: , MicroMod_ATP_CarrierBoard:#I2S_CLK#5
- removed U$53: , MicroMod_ATP_CarrierBoard:#DAT2#5178039
- removed U$54: , MicroMod_ATP_CarrierBoard:#CIPO1#5178039
- removed U$55: , MicroMod_ATP_CarrierBoard:22229
- removed U$56: , MicroMod_ATP_CarrierBoard:##CIPO1##DAT0#5178038
- removed U$57, U$75: , MicroMod_ATP_CarrierBoard:#COPI1#2
- removed U$59: , MicroMod_ATP_CarrierBoard:##CS##0
- removed U$6, U$98: , MicroMod_ATP_CarrierBoard:#D0#0
- removed U$62: , MicroMod_ATP_CarrierBoard:ATP0
- removed U$63, U$76: , MicroMod_ATP_CarrierBoard:#RX2#3
- removed U$64, U$80: , MicroMod_ATP_CarrierBoard:#TX2#2
- removed U$65, U$78: , MicroMod_ATP_CarrierBoard:#SCL1#3
- removed U$66, U$79: , MicroMod_ATP_CarrierBoard:#SDA1#3
- removed U$67, U$77: , MicroMod_ATP_CarrierBoard:#SCK1#2
- removed U$68: , MicroMod_ATP_CarrierBoard:VIN3
- removed U$69: , MicroMod_ATP_CarrierBoard:3V34
- removed U$71: , MicroMod_ATP_CarrierBoard:I2C4
- removed U$72: , MicroMod_ATP_CarrierBoard:I2C14
- removed U$73: , MicroMod_ATP_CarrierBoard:ATP_CARRIER_BOARD1
- removed U$81: , MicroMod_ATP_CarrierBoard:##CS##5178037
- removed U$82: , MicroMod_ATP_CarrierBoard:#DAT2#5
- removed U$83: , MicroMod_ATP_CarrierBoard:#DAT1#5
- removed U$84: , MicroMod_ATP_CarrierBoard:##CS1##DAT3#5178037
- removed U$85: , MicroMod_ATP_CarrierBoard:#COPI#4
- removed U$86: , MicroMod_ATP_CarrierBoard:#SCK#4
- removed U$87: , MicroMod_ATP_CarrierBoard:#MCLK#6
- removed U$90: , MicroMod_ATP_CarrierBoard:#I2S_FS#7
- removed U$91: , MicroMod_ATP_CarrierBoard:#I2S_CLK#7
- removed U$92: , MicroMod_ATP_CarrierBoard:#RTS#7
- removed U$93: , MicroMod_ATP_CarrierBoard:#CTS#8
- removed U$94: , MicroMod_ATP_CarrierBoard:#TX#9
- removed U$95: , MicroMod_ATP_CarrierBoard:#RX#10
- removed U$96: , MicroMod_ATP_CarrierBoard:#CAN_RX#10
- J3: value CONN_05NO_SILK -> Raspberry_Pi_2_3; footprint MicroMod_ATP_CarrierBoard:1X05_NO_SILK -> Connector_PinSocket_2.54mm:PinSocket_2x20_P2.54mm_Vertical
- moved J3 39.4 mm to (160.7, 81.6)
- moved H3 27.2 mm to (162.0, 129.4)
- moved H1 23.3 mm to (165.8, 80.1)
Connections:
- net /SDA renamed PI_SDA
- J2 pad 2: /SWDIO -> PI_GPIO0
- J2 pad 4: /SWDCK -> PI_GPIO1
- J3 pad 1: /I2C_~{INT} -> +3V3
- J3 pad 2: /SCL -> +5V
- J3 pad 4: 3.3V -> +5V
- J3 pad 5: GND -> PI_SCL
- J6 pad 14: /SCL -> PI_SCL
- J6 pad 16: /I2C_~{INT} -> PI_GPIO9
- J6 pad 20: /RX2 -> PI-SEL
- J6 pad 21: /SWDCK -> PI_GPIO1
- J6 pad 22: /TX2 -> PI-TAD
- J6 pad 23: /SWDIO -> PI_GPIO0
- J6 pad 34: /A0 -> PI-ACT
- J6 pad 38: /A1 -> DBG_LED
- J6 pad 40: /G0 -> PI-D0
- J6 pad 41: /CAN_RXI -> PI-IND
- J6 pad 42: /G1 -> PI-D1
- J6 pad 43: /CAN_TXO -> PI-DTD
- J6 pad 44: /G2 -> PI-D2
- J6 pad 46: /G3 -> PI-D3
- J6 pad 48: /G4 -> PI-D4
- J6 pad 50: /I2S_CLK -> PI-REQ
- J6 pad 52: /I2S_WS -> PI-MSG
- J6 pad 54: /I2S_SDI -> PI-C_D
- J6 pad 56: /I2S_SDO -> PI-I_O
- J6 pad 58: /MCLK -> PI-BSY
- J6 pad 63: /G10/ADC_P -> PI-RST
- J6 pad 65: /G9/ADC_N -> PI-ATN
- J6 pad 67: /G8 -> PI-DP
- J6 pad 69: /G7 -> PI-D7
- J6 pad 71: /G6 -> PI-D6
- J6 pad 73: /G5 -> PI-D5
- J6 pad 8: /G11 -> PI-ACK
- TP2 pad P$1: /SWDIO -> PI_GPIO0
- TP3 pad P$1: /SWDCK -> PI_GPIO1
Routing:
- net 3.3V: track 270.0 -> 151.1 mm, vias 7 -> 5
- net /SDA1: track 85.3 -> 0.00 mm, vias 4 -> 0
- net /SCL1: track 81.3 -> 0.00 mm, vias 2 -> 0
- net /G8: track 76.5 -> 0.00 mm
- net /G7: track 75.7 -> 0.00 mm, vias 2 -> 0
- net /G6: track 73.2 -> 0.00 mm, vias 2 -> 0
- net /G5: track 71.2 -> 0.00 mm, vias 2 -> 0
- net /RX1: track 66.4 -> 0.00 mm, vias 2 -> 0
- net /SCL: track 63.5 -> 0.00 mm
- net /TX1: track 63.5 -> 0.00 mm, vias 2 -> 0
- net /CTS1: track 63.5 -> 0.00 mm, vias 2 -> 0
- net /D1: track 62.9 -> 0.00 mm
- net /D0: track 62.4 -> 0.00 mm, vias 2 -> 0
- net /CAN_TXO: track 62.3 -> 0.00 mm, vias 2 -> 0
- net /CAN_RXI: track 62.1 -> 0.00 mm, vias 2 -> 0
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
Commit message: did some stuff
Parts:
- removed D1: 3.3V, MicroMod_ATP_CarrierBoard:SOD-323
- removed FD1, FD2, FD3, FD4: FIDUCIALUFIDUCIAL, MicroMod_ATP_CarrierBoard:FIDUCIAL-MICRO
- removed H1, H2, H3, H4: STAND-OFF, MicroMod_ATP_CarrierBoard:STAND-OFF
- removed LOGO2: QWIIC_LOGO_5MM, MicroMod_ATP_CarrierBoard:QWIIC_5MM
- removed MEAS1: JUMPER-COMBO_2_NC_TRACE, MicroMod_ATP_CarrierBoard:COMBO-JUMPER_2_NC_TRACE
- removed R3: 5.1k, MicroMod_ATP_CarrierBoard:0603
- removed R5: 100k, MicroMod_ATP_CarrierBoard:0603
- removed TP1, TP2, TP3: TEST-POINT3X5, MicroMod_ATP_CarrierBoard:PAD.03X.05
- removed U5: AP7361C-33, MicroMod_ATP_CarrierBoard:UDFN-8
- added H6: MountingHole_Pad, MountingHole:MountingHole_2.7mm_M2.5_Pad_Via, F.Cu at (158.0, 129.0)
- added H7: MountingHole_Pad, MountingHole:MountingHole_2.7mm_M2.5_Pad_Via, F.Cu at (100.0, 129.0)
- added H8: MountingHole_Pad, MountingHole:MountingHole_2.7mm_M2.5_Pad_Via, F.Cu at (100.0, 80.0)
- added H9: MountingHole_Pad, MountingHole:MountingHole_2.7mm_M2.5_Pad_Via, F.Cu at (158.0, 80.0)
- added J5: Conn_01x03_Male, Connector_PinHeader_2.54mm:PinHeader_1x03_P2.54mm_Vertical, B.Cu at (130.2, 111.7)
- added J7: Conn_01x20_Male, Connector_PinHeader_1.00mm:PinHeader_1x24_P1.00mm_Vertical, B.Cu at (146.9, 109.2)
- added U1: AMS1117-3.3, Package_TO_SOT_SMD:SOT-223-3_TabPin2, F.Cu at (112.3, 116.6)
- 3V3_LED1, VIN_LED1: footprint MicroMod_ATP_CarrierBoard:SMT-JUMPER_2_NC_TRACE_SILK -> Jumper:SolderJumper-2_P1.3mm_Bridged_RoundedPad1.0x1.5mm
- BYP1, EN1: footprint MicroMod_ATP_CarrierBoard:SMT-JUMPER_2_NO_SILK -> Jumper:SolderJumper-2_P1.3mm_Open_RoundedPad1.0x1.5mm
- C1, C13, C6, C7, R1, R4: footprint MicroMod_ATP_CarrierBoard:0603 -> Capacitor_SMD:C_0805_2012Metric_Pad1.18x1.45mm_HandSolder
- C2: footprint MicroMod_ATP_CarrierBoard:EIA3216 -> Capacitor_SMD:C_1206_3216Metric_Pad1.33x1.80mm_HandSolder
- C5: footprint MicroMod_ATP_CarrierBoard:0603 -> Capacitor_SMD:C_0603_1608Metric_Pad1.08x0.95mm_HandSolder
- D2, D3: value RED -> Green; footprint MicroMod_ATP_CarrierBoard:LED-0603 -> LED_SMD:LED_0805_2012Metric_Pad1.15x1.40mm_HandSolder
- J1: value USB_C_2-LAYER_PADS -> U254-051N-4BH806; footprint MicroMod_ATP_CarrierBoard:USB-C-16P-2LAYER-PADS -> SamacSys_Parts:U254051N4BH806
- J3: moved to B.Cu
- R10, R9: footprint MicroMod_ATP_CarrierBoard:0603 -> Resistor_SMD:R_0805_2012Metric_Pad1.20x1.40mm_HandSolder
- R2: value 5.1k -> 0; footprint MicroMod_ATP_CarrierBoard:0603 -> Resistor_SMD:R_0805_2012Metric_Pad1.20x1.40mm_HandSolder
- S1, S2: footprint MicroMod_ATP_CarrierBoard:TACTILE_SWITCH_SMD_5.2MM -> Button_Switch_THT:SW_PUSH_6mm
- moved R8 42.0 mm to (145.6, 126.7)
- moved BT1 42.0 mm to (150.7, 129.4)
- moved D6 42.0 mm to (145.6, 128.4)
- moved D7 42.0 mm to (145.6, 130.0)
- moved LOGO1 41.9 mm to (134.8, 130.2)
- moved H5 33.6 mm to (129.7, 121.7), turned to -90 degrees
- moved VIN_LED1 29.2 mm to (104.8, 129.6)
- moved 3V3_LED1 28.1 mm to (104.8, 127.0)
- moved EN1 26.1 mm to (119.5, 102.4)
- moved BYP1 16.3 mm to (103.8, 103.3)
- moved D2 13.3 mm to (98.7, 122.6)
- moved D3 13.3 mm to (98.7, 124.7)
- moved J1 12.8 mm to (98.9, 114.4)
- moved C13 10.2 mm to (106.3, 109.9), turned to -90 degrees
- moved R2 9.69 mm to (107.3, 120.5), turned to 90 degrees
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Connections:
- R1 pad 1: Net-(D2-PadA) -> Net-(R1-Pad1)
- R2 pad 2: Net-(J1-PadA5) -> Net-(J1-Pad4)
- R4 pad 1: Net-(D3-PadA) -> Net-(D3-Pad2)
- VIN_LED1 pad 1: Net-(D3-PadC) -> Net-(VIN_LED1-Pad1)
Routing:
- net 3.3V: track 151.1 -> 0.00 mm, vias 5 -> 0
- net PI-BSY: track 0.00 -> 62.2 mm, vias 0 -> 3
- net VIN: track 55.4 -> 1.47 mm, vias 2 -> 0
- net PI_SDA: track 0.00 -> 52.9 mm, vias 0 -> 3
- net PI-D3: track 0.00 -> 52.3 mm, vias 0 -> 3
- net PI_SCL: track 0.00 -> 51.9 mm, vias 0 -> 3
- net /~{RESET}: track 50.2 -> 0.00 mm, vias 3 -> 0
- net PI-ATN: track 0.00 -> 47.7 mm, vias 0 -> 3
- net PI-RST: track 0.00 -> 46.9 mm, vias 0 -> 3
- net PI-D6: track 0.00 -> 46.6 mm, vias 0 -> 3
- net PI-D2: track 0.00 -> 45.5 mm, vias 0 -> 3
- net PI-ACT: track 0.00 -> 44.2 mm, vias 0 -> 3
- net PI-ACK: track 0.00 -> 42.7 mm, vias 0 -> 2
- net PI-D1: track 0.00 -> 38.1 mm, vias 0 -> 3
- net PI-SEL: track 0.00 -> 38.1 mm, vias 0 -> 3
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- removed copper zone on F.Cu, net Net-(MEAS1-Pad1)
- removed copper zone on F.Cu, net VIN
Other:
- board size 86.4 x 55.9 mm -> 65 x 56 mm

Commit message: more routing
Routing:
- net VIN: track 1.47 -> 70.1 mm, vias 0 -> 2
- net 3.3V: track 0.00 -> 42.2 mm, vias 0 -> 1
- net /USB_P: track 0.00 -> 39.3 mm, vias 0 -> 2
- net /USB_N: track 0.00 -> 39.2 mm, vias 0 -> 2
- net /RX1: track 0.00 -> 15.1 mm, vias 0 -> 3
- net V_USB: track 3.47 -> 16.0 mm
- net Net-(J1-Pad4): track 0.00 -> 10.8 mm, vias 0 -> 2
- net Net-(3V3_LED1-Pad1): track 0.00 -> 9.59 mm
- net Net-(VIN_LED1-Pad1): track 0.00 -> 8.84 mm
- net /RTS1: track 0.00 -> 8.59 mm, vias 0 -> 1
- net GND: track 5.18 -> 13.2 mm, vias 0 -> 3
- net /D1: track 0.00 -> 5.39 mm, vias 0 -> 1
- net /VIN/3: track 0.00 -> 2.05 mm
- net Net-(R1-Pad1): track 0.00 -> 1.74 mm
- net Net-(D3-Pad2): track 0.00 -> 1.74 mm
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